File: UccMicroDuino/UccMicroDuino.kicad_pcb (KiCad board)
At the start: 2 copper layers, 45 x 45 mm, 14 parts, among them J1 Pcb USB Type A, J2 Header, U1 ATtiny85-20SU

Commit message: 1011641-mi primer versionado con gitBash
Parts:
- moved R2 2.24 mm to (188.5, 90.0), turned to 90 degrees
Routing:
- net Net-(D2-K): track 28.7 -> 31.1 mm
- net Net-(J2-Pin_7): track 38.4 -> 37.1 mm
Changed lines of the file:
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@@
 		)
 		(fp_text user "UCC - uDuino"
-			(at -2.54 -5.08 0)
+			(at 35.3 5.5 0)
 			(layer "F.SilkS")
 			(effects
 				(font
 					(size 0.38608 0.38608)
-					(thickness 0.032512)
+					(thickness 0.077216)
+					(bold yes)
 				)
 				(justify left bottom)
@@
 	(footprint "Resistor_SMD:R_0805_2012Metric_Pad1.20x1.40mm_HandSolder"
 		(layer "F.Cu")
-		(at 187.5 92)
+		(at 188.5 90 90)
 		(descr "Resistor SMD 0805 (2012 Metric), square (rectangular) end terminal, IPC-7351 nominal with elongated pad for handsoldering. (Body size source: IPC-SM-782 page 72, https://www.pcb-3d.com/wordpress/wp-content/uploads/ipc-sm-782a_amendment_1_and_2.pdf), generated with kicad-footprint-generator")
 		(tags "resistor handsolder")
 		(property "Reference" "R2"
-			(at 0 -1.65 0)
+			(at 0 -1.65 90)
 			(layer "F.SilkS")
 			(effects
@@
 		)
 		(property "Value" "68Ω 5% 1/8W"
-			(at 0 1.65 0)
+			(at 0 1.65 90)
 			(layer "F.Fab")
 			(effects
@@
 		)
 		(property "Datasheet" "~"
-			(at 0 0 0)
+			(at 0 0 90)
 			(layer "F.Fab")
 			(hide yes)
@@
 		)
 		(property "Description" ""
-			(at 0 0 0)
+			(at 0 0 90)
 			(layer "F.Fab")
 			(hide yes)
@@
 		)
 		(fp_text user "${REFERENCE}"
-			(at 0 0 0)
+			(at 0 0 90)
 			(layer "F.Fab")
 			(effects
@@
 		)
 		(pad "1" smd roundrect
-			(at -1 0)
+			(at -1 0 90)
 			(size 1.2 1.4)
 			(layers "F.Cu" "F.Mask" "F.Paste")
@@
 		)
 		(pad "2" smd roundrect
-			(at 1 0)
+			(at 1 0 90)
 			(size 1.2 1.4)
 			(layers "F.Cu" "F.Mask" "F.Paste")
@@
 	)
 	(segment
-		(start 188.5 92)
-		(end 191.445852 92)
-		(width 0.6)
-		(layer "F.Cu")
-		(net "Net-(J2-Pin_7)")
-	)
-	(segment
 		(start 212.5 93.3)
 		(end 206.531 87.331)
@@
 	)
 	(segment
+		(start 200.484172 82.972926)
+		(end 194.527074 82.972926)
+		(width 0.6)
+		(layer "F.Cu")
+		(net "Net-(J2-Pin_7)")
+	)
+	(segment
 		(start 203.762696 81.478549)
 		(end 201.978549 81.478549)
@@
 	)
 	(segment
-		(start 200.472927 82.972926)
-		(end 200.484172 82.972926)
-		(width 0.6)
-		(layer "F.Cu")
-		(net "Net-(J2-Pin_7)")
-	)
-	(segment
 		(start 203.892073 81.607927)
 		(end 203.762696 81.478549)
@@
 	)
 	(segment
-		(start 191.445852 92)
-		(end 200.472927 82.972926)
-		(width 0.6)
-		(layer "F.Cu")
-		(net "Net-(J2-Pin_7)")
-	)
-	(segment
 		(start 200.484172 82.972926)
 		(end 201.978549 81.478549)
@@
 	)
 	(segment
+		(start 194.527074 82.972926)
+		(end 188.5 89)
+		(width 0.6)
+		(layer "F.Cu")
+		(net "Net-(J2-Pin_7)")
+	)
+	(segment
 		(start 206.531 84.246853)
 		(end 203.892073 81.607927)
@@
 	)
 	(segment
+		(start 188.5 91)
+		(end 187.5 91)
+		(width 0.6)
+		(layer "F.Cu")
+		(net "Net-(D2-K)")
+	)
+	(segment
 		(start 186.5 103)
 		(end 184 105.5)
@@
 		(width 0.6)
 		(layer "F.Cu")
+		(net "Net-(D2-K)")
+	)
+	(segment
+		(start 187.5 91)
+		(end 186.5 92)
+		(width 0.6)
+		(layer "F.Cu")
